Commit message: modifications to driver for remote serial on urXe robots - use instead of the URScript implementation

File: robotiq_85_description/urdf/robotiq_85_gripper_non_root.xacro (robot description, xacro)
@@ -3,6 +3,6 @@
     <xacro:include filename="$(find robotiq_85_description)/urdf/robotiq_85_gripper.urdf.xacro" />
     <link name="gripper_root_link"/>
-    <xacro:robotiq_85_gripper prefix="" parent="gripper_root_link" >
-        <origin xyz="0.05 0 0.85" rpy="0 0 0"/>
+    <xacro:robotiq_85_gripper prefix="" parent="gripper_root_link">
+        <origin xyz="0 0 0" rpy="0 0 0"/>
     </xacro:robotiq_85_gripper>
 </robot>
